File: PCB/SBC_rev 3.sch (EAGLE design)
At the start: 47 parts, among them IC1 74ALS00D, IC2 74LS138D, IC4 PCA9534D, IC5 PCA9534D, IC6 PCA9534D, IC7 74LS32D

Commit message: Updates
Parts:
- added /ATMEL, INT, RD, WR: TPB1,27, testpad:TPB1,27
- added C3, C4, C5, C6: .1uf, zx_kit2:RESISTOR_C-US025-024X044
- added C7: 100uf, adafruit:CPOL-USE2.5-7
- added C8: 1uf, zx_kit2:RESISTOR_C-US025-024X044
- added JP3: (no value), pinhead:PINHD-1X2/90
- added ON: (no value), adafruit:LED3MM
- added R13, R14, R16, R17, R18: 10k, rcl:R-US_R1206
- added R15: 1k, rcl:R-US_R1206
- added RST: PROG, adafruit:PINHD-1X1
- JP1: value KEYRX -> KEY
- JP2: value EXTCLK -> FASTCLK
- renumbered U$15 to SD_ADAPTER
Connections:
- removed net N$27: IC8.M1
- removed net N$3: U$1.P$41
- removed net _MCU_VBUS: U$2.VBUS
- new net M1: IC8.M1, U$1.P$33
- new net N$1: IC1D.I0
- new net N$2: IC1D.I1
- new net N$7: ON.A, R15.2
- new net TIMER4: JP2.1, U$2.PC7(ICP3/CLK0/OC4A)
- net /ATMELSERIAL: now also /ATMEL.TP
- net FASTCLK: now also IC1A.I1, JP2.2, U$1.P$22; no longer JP2.1, U$2.PC7(ICP3/CLK0/OC4A)
- net GND: now also C3.2, C4.2, C5.2, C6.2, C7.-, C8.2, JP3.2, ON.C
- net INT: now also INT.TP
- net KEYBOARD_RX: now also R16.1
- net MCU_RST: now also RST.1; no longer U$1.P$33
- net N$6: now also IC1D.O; no longer IC1A.I1, JP2.2
- net NMI: now also R18.1
- net RD: now also RD.TP
- net SCL: now also R14.1
- net SDA: now also R13.1
- net UCAP: now also C8.1
- net VBUS: now also JP3.1
- net VCC: now also C3.1, C4.1, C5.1, C6.1, C7.+, R13.2, R14.2, R15.1, R16.2, R17.2, R18.2, U$2.VBUS
- net WAIT: now also R17.1
- net WR: now also WR.TP
- net Z80CLK: now also U$1.P$41; no longer U$1.P$22
Other:
- moved on the sheet: C1, C2, R10, R5
